File: Hardware/Sim_Breakout.brd (EAGLE design)
At the start: 25.4 x 31.2 mm, 7 parts, among them U2 SIMHOLDER

Commit message: Aesthetic changes
1. Updated net labels to flags.
2.) Added OSHW logo to bottom silk.
3.) Added SFE logo to bottom silk.
Parts:
- added LOGO1: OSHW-LOGOS, SparkFun-Aesthetics:OSHW-LOGO-S
- added U$1: (no value), SparkFun-Aesthetics:SFE-NEW-WEBLOGO
- moved FRAME2 42.6 mm to (-19.1, -10.2)
Changed lines of the file:
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@@
 <setting verticaltext="up"/>
 </settings>
-<grid distance="0.05" unitdist="inch" unit="inch" style="lines" multiple="1" display="yes" altdistance="0.01" altunitdist="inch" altunit="inch"/>
+<grid distance="0.05" unitdist="inch" unit="inch" style="lines" multiple="1" display="yes" altdistance="0.005" altunitdist="inch" altunit="inch"/>
 <layers>
 <layer number="1" name="Top" color="4" fill="1" visible="yes" active="yes"/>
@@
 <layer number="19" name="Unrouted" color="6" fill="1" visible="yes" active="yes"/>
 <layer number="20" name="Dimension" color="6" fill="1" visible="yes" active="yes"/>
-<layer number="21" name="tPlace" color="6" fill="1" visible="yes" active="yes"/>
-<layer number="22" name="bPlace" color="6" fill="1" visible="yes" active="yes"/>
+<layer number="21" name="tPlace" color="16" fill="1" visible="yes" active="yes"/>
+<layer number="22" name="bPlace" color="14" fill="1" visible="yes" active="yes"/>
 <layer number="23" name="tOrigins" color="15" fill="1" visible="yes" active="yes"/>
 <layer number="24" name="bOrigins" color="15" fill="1" visible="yes" active="yes"/>
@@
 <text x="12.446" y="-1.016" size="0.4064" layer="27">SIM Socket Opening this end</text>
 <text x="22.606" y="13.208" size="0.4064" layer="27" rot="R90">No leads soldered to these pads</text>
-<text x="10.541" y="24.384" size="1.778" layer="22" font="vector" ratio="15" rot="MR270">SIM Breakout</text>
+<text x="12.192" y="24.003" size="1.778" layer="22" font="vector" ratio="15" rot="MR270">SIM Breakout</text>
 <text x="6.096" y="23.495" size="1.27" layer="22" ratio="15" rot="MR0">VCC</text>
 <text x="6.096" y="20.955" size="1.27" layer="22" ratio="15" rot="MR0">RST</text>
@@
 <text x="6.096" y="5.715" size="1.27" layer="22" ratio="15" rot="MR0">GND</text>
 <text x="24.13" y="29.718" size="1.016" layer="16" font="vector" ratio="25" rot="MR0">v13</text>
-<text x="52.07" y="-22.86" size="1.778" layer="51" font="vector" ratio="7">Robert Hunke</text>
+<text x="11.43" y="-10.16" size="1.778" layer="51" font="vector" ratio="7">Robert Hunke</text>
 </plain>
 <attributes>
@@
 <element name="STANDOFF1" library="SparkFun-Electromechanical" package="STAND-OFF" value="STAND-OFF" x="3.81" y="27.94"/>
 <element name="STANDOFF2" library="SparkFun-Electromechanical" package="STAND-OFF" value="STAND-OFF" x="3.81" y="2.54"/>
-<element name="FRAME2" library="SparkFun-Aesthetics" package="CREATIVE_COMMONS" value="FRAME-LETTER" x="21.59" y="-22.86"/>
+<element name="FRAME2" library="SparkFun-Aesthetics" package="CREATIVE_COMMONS" value="FRAME-LETTER" x="-19.05" y="-10.16"/>
 <element name="FID1" library="SparkFun-Aesthetics" package="MICRO-FIDUCIAL" value="FIDUCIALUFIDUCIAL" x="1.016" y="1.27"/>
 <element name="FID2" library="SparkFun-Aesthetics" package="MICRO-FIDUCIAL" value="FIDUCIALUFIDUCIAL" x="6.35" y="30.48"/>
+<element name="LOGO1" library="SparkFun-Aesthetics" package="OSHW-LOGO-S" value="OSHW-LOGOS" x="22.86" y="2.54" rot="MR90"/>
+<element name="U$1" library="SparkFun-Aesthetics" package="SFE-NEW-WEBLOGO" value="" x="14.605" y="5.588" rot="MR90"/>
 </elements>
 <signals>
